File: modem.kicad_sch (KiCad schematic)
At the start: 17 parts, among them J1 Conn_01x05_Pin, J3 Conn_01x02_Pin, Y1 Crystal_Small

Commit message: Improved docs
Other:
- note added: "Connection to Loop Transformer"
- note added: "Control Lines"
- company: (none) -> Bruce MacKinnon
- title: (none) -> Bell 103 Host - Modem Sheet
Changed lines of the file:
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@@
 (kicad_sch (version 20230121) (generator eeschema)
   (paper "A4")
+  (title_block
+    (title "Bell 103 Host - Modem Sheet")
+    (date "2023-08-20")
+    (rev "v1")
+    (company "Bruce MacKinnon")
+  )
   (junction (at 179.07 85.09) (diameter 0) (color 0 0 0 0)
   )
@@
     (stroke (width 0) (type default))
   )
+  (text "Connection to Loop Transformer" (at 148.59 123.19 0)
+    (effects (font (size 1.27 1.27)) (justify left bottom))
+  )
+  (text "Control Lines" (at 161.29 53.34 0)
+    (effects (font (size 1.27 1.27)) (justify left bottom))
+  )
   (global_label "RXAN" (shape input) (at 113.03 90.17 180) (fields_autoplaced)
