File: subscriber-loop.kicad_sch (KiCad schematic)
At the start: 13 parts, among them J4 Conn_01x02, J5 Conn_01x01, J6 Conn_01x02, J7 Conn_01x01, Q1 MMBT3904, T1 Transformer_1P_1S

Commit message: Improved docs
Other:
- note added: "Subscriber Loop"
- note removed: "Subscriber Line"
- company: (none) -> Bruce MacKinnon
- title: (none) -> Bell 103 Host - Subscriber Loop Sheet
Changed lines of the file:
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@@
 (kicad_sch (version 20230121) (generator eeschema)
   (paper "A4")
+  (title_block
+    (title "Bell 103 Host - Subscriber Loop Sheet")
+    (date "2023-08-20")
+    (rev "v1")
+    (company "Bruce MacKinnon")
+  )
   (junction (at 99.06 48.26) (diameter 0) (color 0 0 0 0)
   )
@@
     (effects (font (size 1.27 1.27)) (justify left bottom))
   )
-  (text "Subscriber Line" (at 100.33 68.58 0)
+  (text "Subscriber Loop " (at 100.33 68.58 0)
     (effects (font (size 1.27 1.27)) (justify left bottom))
   )
